File: pcb/pcb_power/pcb_power.kicad_sch (KiCad schematic)
At the start: 3 parts, among them J10 Conn_01x04, J11 Conn_01x04, J40 XT30

Commit message: fin board
Parts:
- J10: value Conn_01x04 -> JST_B4B-XH-A
- J11: value Conn_01x04 -> JST_B4P-VH; footprint Connector_JST:JST_VH_B4P-VH-FB-B_1x04_P3.96mm_Vertical -> Connector_JST:JST_VH_B4P-VH_1x04_P3.96mm_Vertical
- renumbered J40 to J12
Connections:
- net Tab selector/Relay_GND is gone; now on net Tab selector/Relay1: J10.1 (Pin_1)
- net Rectifier/AC1: now also J11.4 (Pin_4); no longer J11.1 (Pin_1)
- net Tab selector/10V_AC: now also J11.3 (Pin_3); no longer J11.2 (Pin_2)
- net Tab selector/20V_AC: now also J11.2 (Pin_2); no longer J11.3 (Pin_3)
- net Tab selector/30V_AC: now also J11.1 (Pin_1); no longer J11.4 (Pin_4)
- net Tab selector/Relay1: no longer J10.2 (Pin_2)
- net Tab selector/Relay2: now also J10.2 (Pin_2); no longer J10.3 (Pin_3)
- new net Tab selector/Relay_VCC: J10.3 (Pin_3)
Other:
- sheet Tab selector ports: added Relay_VCC; removed Relay_GND
