File: pcb/pcb_power/rectifier.kicad_sch (KiCad schematic)
At the start: 6 parts

Commit message: fin board
Parts:
- C30, C31: footprint Capacitor_THT:CP_Radial_D14.0mm_P7.50mm -> Capacitor_THT:CP_Radial_D22.0mm_P10.00mm_SnapIn
- renumbered D1 to D30, D3 to D31, D2 to D32, D4 to D33
Other:
- note added: "30V 5A Linear Power Supply"
