File: pcb/pcb_controller/pcb_controller.kicad_sch (KiCad schematic)
At the start: 5 parts, among them J10 Conn_01x04, J103 Banana conn, J103 JST_XH_B3B-XH, J104 JST_XH_B2B-XH, J104 XT30

Commit message: most analog layout
Parts:
- J10: value Conn_01x04 -> JST_XH_B4B-XH
Connections:
- net +12V: now also J10.3 (Pin_3)
- net MCU/relay1: now reaches J10.1 (Pin_1)
- net MCU/relay2: now reaches J10.2 (Pin_2)
Other:
- sheet MCU ports: added +Vout_sense, -Vout_sense, I_set, U_set, relay1, relay2; removed none
- moved on the sheet: J10, J103

Commit message: minor changes
Connections:
- net GNDREF renamed EARTH
Changed lines of the file:
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@@
 			)
 		)
-		(property "Value" "GNDREF"
+		(property "Value" "EARTH"
 			(at 158.75 38.1 0)
 			(effects
