File: pcb/pcb_controller/power.kicad_sch (KiCad schematic)
At the start: 15 parts, among them U201 MC78L05, U202 MC79L05

Commit message: minor changes
Other:
- company: (none) -> Dominik Workshop
Changed lines of the file:
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@@
 	(generator_version "8.0")
 	(paper "A5")
+	(title_block
+		(rev "V1.0")
+		(company "Dominik Workshop")
+	)
 	(junction
 		(at 133.35 39.37)
